File: boards/flashpi.kicad_pcb (KiCad board)
At the start: 2 copper layers, 65 x 56.5 mm, 16 parts, among them J1 RPi_GPIO_Compact, SW1 WRITE_PROTECT, SW2 POWER

Commit message: Deploying to gh-pages from @ neg2led/flashpi@cf96e1e5e2df5559336897a5176b93a9f1f65f92 🚀
Parts:
- moved SW1 51.4 mm to (176.6, 88.1), turned to 270 degrees
- moved LOGO1 10.7 mm to (137.3, 117.2), turned to 180 degrees
- moved C1 0.50 mm to (169.2, 97.8)
- moved C2 0.50 mm to (158.8, 112.7)
- moved C3 0.50 mm to (137.8, 98.8)
- moved C4 0.50 mm to (133.8, 109.5)
- moved H1 0.50 mm to (121.0, 75.5)
- moved H2 0.50 mm to (179.0, 75.5)
- moved H3 0.50 mm to (121.0, 124.5)
- moved H4 0.50 mm to (179.0, 124.5)
- moved I2C1 0.50 mm to (137.2, 105.0)
- moved J1 0.50 mm to (150.0, 75.5)
- moved JI2C1 0.50 mm to (133.4, 89.5)
- moved JSPI1 0.50 mm to (158.7, 89.5)
- moved SPI1 0.50 mm to (162.5, 107.0)
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Routing:
- net Board_1-VCC: track 187.7 -> 62.4 mm
- net Board_1-/SPI_WP: track 64.2 -> 0.37 mm, vias 2 -> 0
- net Board_1-/I2C_WP: track 50.0 -> 2.45 mm, vias 1 -> 0
- net Board_1-/~SPI_CS: track 50.2 -> 13.3 mm
- net Board_1-/SPI_MOSI: track 64.2 -> 28.2 mm, vias 2 -> 1
- net Board_1-/SPI_CLK: track 55.5 -> 22.0 mm
- net Board_1-/SPI_MISO: track 50.3 -> 18.0 mm
- net Board_1-/I2C_SDA: track 56.3 -> 26.5 mm, vias 1 -> 0
- net Board_1-/I2C_SCL: track 53.4 -> 26.8 mm
- net Board_1-GND: vias 31 -> 19
